File: Hardware/RedBoard.sch (EAGLE design)
At the start: 65 parts, among them IC3 LM1117, J2 ICSP, J3 POWER_JACKSUPER_BOMB_DIGITY, Q1 1A/60V/500mΩ, Q2 2N7002PW, U1 FT231XS, U2 MIC5205, U4 ATMEGA328P_TQFP, Y1 16MHz

Commit message: Initial commit.
Changed USB. Added Qwiic. Added I/O jumper.
Parts:
- removed C13, C9: 47pF, SparkFun-Capacitors:47PF-0603-50V-5%
- removed C14: 0.1uF, SparkFun-Capacitors:0.1UF-0603-25V-(+80/-20%)
- removed FRAME2: FRAME-LETTER, SparkFun-Aesthetics:FRAME-LETTER
- removed JP12: USB-MINIB-5PIN, SparkFun-Connectors:USB-MINIB-5PIN
- removed LED3: Red, SparkFun-LED:LED1206
- removed LED4: Yellow, SparkFun-LED:LED1206
- removed R10: 27, SparkFun-Resistors:27OHM-0603-1/10W-1%
- removed R7, R8, R9: 1k, SparkFun-Resistors:1KOHM-0603-1/10W-1%
- removed U1: FT231XS, SparkFun-IC-Comms:FT231XS
- added C11: 22pF, SparkFun-Capacitors:22PF-0603-50V-5%
- added C16: 1.0uF, SparkFun-Capacitors:1.0UF-16V-10%(0603)
- added C17: 10nF, SparkFun-Capacitors:10NF/10000PF-50V-10%(0603)
- added C18: 0.1uF, SparkFun-Capacitors:0.1UF-25V(+80/-20%)(0603)
- added D3: Yellow, SparkFun-LED:LED-YELLOW_HIDDENSILK
- added FRAME1: FRAME-LEDGER, SparkFun-Aesthetics:FRAME-LEDGER
- added I/O: JUMPER-SMT_3_1-NC_TRACE_SILK, SparkFun-Jumpers:JUMPER-SMT_3_1-NC_TRACE_SILK
- added J1: microB, SparkFun-Connectors:USB_MICRO-B_HALF_PTH
- added J4: SMD, SparkX:I2C_STANDARDJS-1MM
- added LED5: GREEN, SparkFun-LED:LED-GREEN_HIDDENSILK
- added Q3: 2N7002PW, SparkFun-DiscreteSemi:MOSFET-NCH-2N7002PW
- added R12: 1K, SparkFun-Resistors:1KOHM-1/10W-1%(0603)
- added R16: 330, SparkFun-Resistors:330OHM1/10W1%(0603)
- added U3: AP2112-3.3V, SparkFun-PowerIC:V_REG_AP2112K-3.3V
- added Y2: 12MHz, USB Basic:CRYSTAL-GROUNDED3.2X2.5
- C7: value 1.0uF -> 22pF; device SparkFun-Capacitors:1.0UF-0603-16V-10% -> SparkFun-Capacitors:22PF-0603-50V-5%
- F1: value 6V/0.5A -> PPTC_6V500MA; device SparkFun-Fuses:PTC-HALF_AMP -> SparkFun-Fuses:PPTC_6V500MA
- JP10: value JP10 -> (none)
- JP11: value IOL -> JP11
- JP13: value AD -> (none)
- LED1: device SparkFun-LED:LED1206 -> SparkFun-LED:LED-BLUE_HIDDENSILK
- LED2: value Green -> GREEN; device SparkFun-LED:LED1206 -> SparkFun-LED:LED-GREEN_HIDDENSILK
- R11, R13: value 10k -> 2.2k; device SparkFun-Resistors:10KOHM-0603-1/10W-1% -> SparkFun-Resistors:2.2KOHM-0603-1/10W-1%
- R5: value 27 -> 2.2k; device SparkFun-Resistors:27OHM-0603-1/10W-1% -> SparkFun-Resistors:2.2KOHM-0603-1/10W-1%
- R6: value 1k -> 2.2k; device SparkFun-Resistors:1KOHM-0603-1/10W-1% -> SparkFun-Resistors:2.2KOHM-0603-1/10W-1%
- U2: value MIC5205 -> CH340G; device SparkFun-PowerIC:MIC52053.3V -> SparkFun-DigitalIC:CH340GSMD
Connections:
- removed net 3.3V_F: C14.1, Q2.G, R11.2, U1.!RESET, U1.3V3OUT, U1.VCCIO
- removed net D+: C9.1, JP12.D+, R10.1
- removed net D-: C13.1, JP12.D-, R5.1
- removed net DTR: C8.1, Q2.D, R13.1
- removed net FTDI_DTR: Q2.S, R11.1, U1.!DTR
- removed net N$10: LED4.A, R7.2
- removed net N$6: R5.2, U1.USBDM
- removed net N$7: R10.2, U1.USBDP
- removed net N$8: LED3.A, R6.2
- removed net RXD: R9.2, U1.RXD
- removed net RXLED: LED4.C, U1.CBUS1
- removed net TXD: R8.2, U1.TXD
- removed net TXLED: LED3.C, U1.CBUS2
- new net !DTR: C8.1, U2.!DTR
- new net LV_SCL: J4.SCL, Q2.S, R11.1
- new net LV_SDA: J4.SDA, Q3.S, R5.1
- new net N$11: C11.2, U2.XO, Y2.2
- new net N$12: C7.2, U2.XI, Y2.1
- new net N$13: J1.D-, U2.UD-
- new net N$14: J1.D+, U2.UD+
- new net N$5: LED5.A, R16.1
- new net N$9: D3.A, R12.1
- new net SHLD: J1.SHIELD
- new net V3: C17.1, U2.V3
- new net VCC: C18.1, C2.2, I/O.2, J2.2, R12.2, R13.2, R16.2, R2.2, R3.2, R6.2, TP1.1, U2.VCC, U4.AVCC, U4.VCC@4, U4.VCC@6
- net 3.3V: now also C16.1, I/O.1, J4.VCC, Q2.G, Q3.G, R11.2, R5.2, U3.OUT; no longer C7.1, U2.OUT
- net 5V: now also I/O.3, U3.EN, U3.IN; no longer C2.2, J2.2, R13.2, R2.2, R3.2, R6.1, R7.1, TP1.1, U2.EN, U2.IN, U4.AVCC, U4.VCC@4, U4.VCC@6
- net AD4/SDA: now also Q3.D, R6.1
- net AD5/SCL: now also Q2.D, R13.1
- net GND: now also C11.1, C16.2, C17.2, C18.2, C7.1, J1.GND, J4.GND, U3.GND, Y2.GND; no longer C13.2, C14.2, C7.2, C9.2, JP12.GND, JP12.MTN1, JP12.MTN2, JP12.MTN3, JP12.MTN4, U1.GND@16, U1.GND@6
- net RX-I: now also D3.C, U2.TXD; no longer R8.1
- net TX-O: now also LED5.C, U2.RXD; no longer R9.1
- net USBVCC: no longer U1.VCC
- net VUSB: now also J1.VBUS; no longer JP12.VBUS
Other:
- note added: "3.3V 600mA Out"
- note added: "3.3V Regulation"
- note added: "Board I/O Voltage"
- note added: "Green LED is very dim on Serial Basic. Will larger 1206 LED be brighter with 330?"
- note added: "Jim Lindblom, N. Seidle"
- note added: "Keep power LED as green?"
- note added: "Qwiic"
- note added: "To convert the board to 3.3V you must cut the jumper to 5V and use solder to close the jumper towards 3.3V."
- note added: "USB-to-Serial Converter"
- note added: "red for power, blue for STAT, green for TX, yellow for RX"
- note added: "v23"
- note removed: "3.3V 150mA Out"
- note removed: "FT231XS (USB-to-Serial Converter)"
- note removed: "Jim Lindblom"
- note removed: "v22"
- moved on the sheet: C1, C10, C12, C15, C2, C3, C4, C5, C6, C7, C8, D1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
